Commit message: new sensor - falcon lidar

File: golfcart_sensor_kit_description/urdf/sensor_kit.xacro (robot description, xacro)
@@ -16,5 +16,5 @@
     <!-- sensor -->
     <xacro:property name="calibration" value="${xacro.load_yaml('$(arg config_dir)/sensor_kit_calibration.yaml')}"/>
-    <!-- lidar -->
+    <!-- VLP lidar -->
     <joint name="lidar_joint" type="fixed">
       <origin
@@ -27,7 +27,27 @@
       />
       <parent link="sensor_kit_base_link"/>
-      <child link="lidar"/>
+      <child link="vlp_lidar"/>
     </joint>
-    <link name="lidar">
+    <link name="vlp_lidar">
+      <inertial>
+        <mass value="0.1"/>
+        <origin xyz="0 0 0"/>
+        <inertia ixx="0.1" ixy="0" ixz="0" iyy="0.1" iyz="0" izz="0.1"/>
+      </inertial>
+    </link>
+    <!-- Falcon lidar -->
+    <joint name="falcon_lidar_joint" type="fixed">
+      <origin
+        xyz="${calibration['sensor_kit_base_link']['falcon']['x']}
+             ${calibration['sensor_kit_base_link']['falcon']['y']}
+             ${calibration['sensor_kit_base_link']['falcon']['z']}"
+        rpy="${calibration['sensor_kit_base_link']['falcon']['roll']}
+             ${calibration['sensor_kit_base_link']['falcon']['pitch']}
+             ${calibration['sensor_kit_base_link']['falcon']['yaw']}"
+      />
+      <parent link="sensor_kit_base_link"/>
+      <child link="falcon_lidar"/>
+    </joint>
+    <link name="falcon_lidar">
       <inertial>
         <mass value="0.1"/>
@@ -76,5 +96,5 @@
       </inertial>
     </link>
-    <!-- TODO: Add USB/Tier IV camera frames when camera integration is ready -->
+    <!-- TODO, Add USB/Tier IV camera frames when camera integration is ready -->
   </xacro:macro>
 </robot>

Commit message: feat: add seyond and cameras to launch file

File: golfcart_sensor_kit_description/urdf/sensor_kit.xacro (robot description, xacro)
@@ -47,7 +47,7 @@
       />
       <parent link="sensor_kit_base_link"/>
-      <child link="falcon_lidar"/>
+      <child link="seyond"/>
     </joint>
-    <link name="falcon_lidar">
+    <link name="seyond">
       <inertial>
         <mass value="0.1"/>
@@ -96,29 +96,44 @@
       </inertial>
     </link>
-    <!-- USB cameras (TIER IV C1 via GMSL2-USB) — placeholder transforms; update after physical mounting -->
-    <xacro:macro name="usb_camera_frame" params="name">
-      <joint name="${name}_joint" type="fixed">
+    <!-- USB/Tier IV camera -->
+    <joint name="camera_left_joint" type="fixed">
         <origin
-          xyz="${calibration['sensor_kit_base_link'][name]['x']}
-               ${calibration['sensor_kit_base_link'][name]['y']}
-               ${calibration['sensor_kit_base_link'][name]['z']}"
-          rpy="${calibration['sensor_kit_base_link'][name]['roll']}
-               ${calibration['sensor_kit_base_link'][name]['pitch']}
-               ${calibration['sensor_kit_base_link'][name]['yaw']}"
-        />
+        xyz="${calibration['sensor_kit_base_link']['usb_camera_left']['x']}
+             ${calibration['sensor_kit_base_link']['usb_camera_left']['y']}
+             ${calibration['sensor_kit_base_link']['usb_camera_left']['z']}"
+        rpy="${calibration['sensor_kit_base_link']['usb_camera_left']['roll']}
+             ${calibration['sensor_kit_base_link']['usb_camera_left']['pitch']}
+             ${calibration['sensor_kit_base_link']['usb_camera_left']['yaw']}"
+            />
         <parent link="sensor_kit_base_link"/>
-        <child link="${name}"/>
-      </joint>
-      <link name="${name}">
-        <inertial>
-          <mass value="0.1"/>
-          <origin xyz="0 0 0"/>
-          <inertia ixx="0.1" ixy="0" ixz="0" iyy="0.1" iyz="0" izz="0.1"/>
-        </inertial>
-      </link>
-    </xacro:macro>
-    <xacro:usb_camera_frame name="usb_camera_left_optical_link"/>
-    <xacro:usb_camera_frame name="usb_camera_right_optical_link"/>
-    <xacro:usb_camera_frame name="usb_camera_rear_optical_link"/>
+        <child link="usb_camera_left"/>
+    </joint>
+    <link name="usb_camera_left"/>
+    <joint name="camera_rear_joint" type="fixed">
+        <origin
+        xyz="${calibration['sensor_kit_base_link']['usb_camera_rear']['x']}
+             ${calibration['sensor_kit_base_link']['usb_camera_rear']['y']}
+             ${calibration['sensor_kit_base_link']['usb_camera_rear']['z']}"
+        rpy="${calibration['sensor_kit_base_link']['usb_camera_rear']['roll']}
+             ${calibration['sensor_kit_base_link']['usb_camera_rear']['pitch']}
+             ${calibration['sensor_kit_base_link']['usb_camera_rear']['yaw']}"
+            />
+        <parent link="sensor_kit_base_link"/>
+        <child link="usb_camera_rear"/>
+    </joint>
+    <link name="usb_camera_rear"/>
+    <joint name="camera_right_joint" type="fixed">
+        <origin
+        xyz="${calibration['sensor_kit_base_link']['usb_camera_right']['x']}
+             ${calibration['sensor_kit_base_link']['usb_camera_right']['y']}
+             ${calibration['sensor_kit_base_link']['usb_camera_right']['z']}"
+        rpy="${calibration['sensor_kit_base_link']['usb_camera_right']['roll']}
+             ${calibration['sensor_kit_base_link']['usb_camera_right']['pitch']}
+             ${calibration['sensor_kit_base_link']['usb_camera_right']['yaw']}"
+            />
+        <parent link="sensor_kit_base_link"/>
+        <child link="usb_camera_right"/>
+    </joint>
+    <link name="usb_camera_right"/>
   </xacro:macro>
 </robot>

Commit message: feat: change from raw to jpg, remove usb_ from name

File: golfcart_sensor_kit_description/urdf/sensor_kit.xacro (robot description, xacro)
@@ -99,41 +99,41 @@
     <joint name="camera_left_joint" type="fixed">
         <origin
-        xyz="${calibration['sensor_kit_base_link']['usb_camera_left']['x']}
-             ${calibration['sensor_kit_base_link']['usb_camera_left']['y']}
-             ${calibration['sensor_kit_base_link']['usb_camera_left']['z']}"
-        rpy="${calibration['sensor_kit_base_link']['usb_camera_left']['roll']}
-             ${calibration['sensor_kit_base_link']['usb_camera_left']['pitch']}
-             ${calibration['sensor_kit_base_link']['usb_camera_left']['yaw']}"
+        xyz="${calibration['sensor_kit_base_link']['camera_left']['x']}
+             ${calibration['sensor_kit_base_link']['camera_left']['y']}
+             ${calibration['sensor_kit_base_link']['camera_left']['z']}"
+        rpy="${calibration['sensor_kit_base_link']['camera_left']['roll']}
+             ${calibration['sensor_kit_base_link']['camera_left']['pitch']}
+             ${calibration['sensor_kit_base_link']['camera_left']['yaw']}"
             />
         <parent link="sensor_kit_base_link"/>
-        <child link="usb_camera_left"/>
+        <child link="camera_left"/>
     </joint>
-    <link name="usb_camera_left"/>
+    <link name="camera_left"/>
     <joint name="camera_rear_joint" type="fixed">
         <origin
-        xyz="${calibration['sensor_kit_base_link']['usb_camera_rear']['x']}
-             ${calibration['sensor_kit_base_link']['usb_camera_rear']['y']}
-             ${calibration['sensor_kit_base_link']['usb_camera_rear']['z']}"
-        rpy="${calibration['sensor_kit_base_link']['usb_camera_rear']['roll']}
-             ${calibration['sensor_kit_base_link']['usb_camera_rear']['pitch']}
-             ${calibration['sensor_kit_base_link']['usb_camera_rear']['yaw']}"
+        xyz="${calibration['sensor_kit_base_link']['camera_rear']['x']}
+             ${calibration['sensor_kit_base_link']['camera_rear']['y']}
+             ${calibration['sensor_kit_base_link']['camera_rear']['z']}"
+        rpy="${calibration['sensor_kit_base_link']['camera_rear']['roll']}
+             ${calibration['sensor_kit_base_link']['camera_rear']['pitch']}
+             ${calibration['sensor_kit_base_link']['camera_rear']['yaw']}"
             />
         <parent link="sensor_kit_base_link"/>
-        <child link="usb_camera_rear"/>
+        <child link="camera_rear"/>
     </joint>
-    <link name="usb_camera_rear"/>
+    <link name="camera_rear"/>
     <joint name="camera_right_joint" type="fixed">
         <origin
-        xyz="${calibration['sensor_kit_base_link']['usb_camera_right']['x']}
-             ${calibration['sensor_kit_base_link']['usb_camera_right']['y']}
-             ${calibration['sensor_kit_base_link']['usb_camera_right']['z']}"
-        rpy="${calibration['sensor_kit_base_link']['usb_camera_right']['roll']}
-             ${calibration['sensor_kit_base_link']['usb_camera_right']['pitch']}
-             ${calibration['sensor_kit_base_link']['usb_camera_right']['yaw']}"
+        xyz="${calibration['sensor_kit_base_link']['camera_right']['x']}
+             ${calibration['sensor_kit_base_link']['camera_right']['y']}
+             ${calibration['sensor_kit_base_link']['camera_right']['z']}"
+        rpy="${calibration['sensor_kit_base_link']['camera_right']['roll']}
+             ${calibration['sensor_kit_base_link']['camera_right']['pitch']}
+             ${calibration['sensor_kit_base_link']['camera_right']['yaw']}"
             />
         <parent link="sensor_kit_base_link"/>
-        <child link="usb_camera_right"/>
+        <child link="camera_right"/>
     </joint>
-    <link name="usb_camera_right"/>
+    <link name="camera_right"/>
   </xacro:macro>
 </robot>
