Commit message: chore: remove AutoSDV sensor refs (Cube1, Robin-W, ZED)
- lidar.launch.xml: remove Cube1 and Robin-W code paths, keep vlp32c only
- sensor_kit.xacro: remove zed_wrapper include and ZED camera joint/macro,
  fix lidar calibration key to use vlp32c instead of nonexistent 'lidar'
- imu.launch.xml: replace MPU9250 driver with Tamagawa placeholder

Co-Authored-By: Claude Sonnet 4.6 (1M context) <noreply@anthropic.com>

File: golfcart_sensor_kit_description/urdf/sensor_kit.xacro (robot description, xacro)
@@ -2,5 +2,4 @@
 <robot xmlns:xacro="http://ros.org/wiki/xacro">
   <xacro:macro name="sensor_kit_macro" params="parent x y z roll pitch yaw">
-    <xacro:include filename="$(find zed_wrapper)/urdf/zed_macro.urdf.xacro"/>
     <xacro:include filename="$(find imu_description)/urdf/imu.xacro"/>
     <xacro:arg name="gpu" default="false"/>
@@ -20,10 +19,10 @@
     <joint name="lidar_joint" type="fixed">
       <origin
-        xyz="${calibration['sensor_kit_base_link']['lidar']['x']}
-             ${calibration['sensor_kit_base_link']['lidar']['y']}
-             ${calibration['sensor_kit_base_link']['lidar']['z']}"
-        rpy="${calibration['sensor_kit_base_link']['lidar']['roll']}
-             ${calibration['sensor_kit_base_link']['lidar']['pitch']}
-             ${calibration['sensor_kit_base_link']['lidar']['yaw']}"
+        xyz="${calibration['sensor_kit_base_link']['vlp32c']['x']}
+             ${calibration['sensor_kit_base_link']['vlp32c']['y']}
+             ${calibration['sensor_kit_base_link']['vlp32c']['z']}"
+        rpy="${calibration['sensor_kit_base_link']['vlp32c']['roll']}
+             ${calibration['sensor_kit_base_link']['vlp32c']['pitch']}
+             ${calibration['sensor_kit_base_link']['vlp32c']['yaw']}"
       />
       <parent link="sensor_kit_base_link"/>
@@ -77,27 +76,5 @@
       </inertial>
     </link>
-    <!-- camera -->
-    <joint name="zedxm_camera_joint" type="fixed">
-      <origin
-        xyz="${calibration['sensor_kit_base_link']['zedxm_camera_link']['x']}
-             ${calibration['sensor_kit_base_link']['zedxm_camera_link']['y']}
-             ${calibration['sensor_kit_base_link']['zedxm_camera_link']['z']}"
-        rpy="${calibration['sensor_kit_base_link']['zedxm_camera_link']['roll']}
-             ${calibration['sensor_kit_base_link']['zedxm_camera_link']['pitch']}
-             ${calibration['sensor_kit_base_link']['zedxm_camera_link']['yaw']}"
-      />
-      <parent link="sensor_kit_base_link"/>
-      <child link="zedxm_camera_link"/>
-    </joint>
-    <xacro:zed_camera name="zedxm" model="zedxm" custom_baseline="0" enable_gnss="false">
-      <origin
-        xyz="${calibration['sensor_kit_base_link']['zedxm_camera_link']['x']}
-             ${calibration['sensor_kit_base_link']['zedxm_camera_link']['y']}
-             ${calibration['sensor_kit_base_link']['zedxm_camera_link']['z']}"
-        rpy="${calibration['sensor_kit_base_link']['zedxm_camera_link']['roll']}
-             ${calibration['sensor_kit_base_link']['zedxm_camera_link']['pitch']}
-             ${calibration['sensor_kit_base_link']['zedxm_camera_link']['yaw']}"
-      />
-    </xacro:zed_camera>
+    <!-- TODO: Add USB/Tier IV camera frames when camera integration is ready -->
   </xacro:macro>
 </robot>

Commit message: feat: add USB camera frames to sensor kit description
Define usb_camera_{left,right,rear}_optical_link frames in sensor_kit.xacro
via a small macro, with placeholder (zero) transforms sourced from
sensor_kit_calibration.yaml. Frame names match the frame_id values the
gscam configs publish; transforms to be filled in after physical mounting.

Co-Authored-By: Claude Opus 4.7 (1M context) <noreply@anthropic.com>

File: golfcart_sensor_kit_description/urdf/sensor_kit.xacro (robot description, xacro)
@@ -27,7 +27,7 @@
       />
       <parent link="sensor_kit_base_link"/>
-      <child link="vlp_lidar"/>
+      <child link="velodyne"/>
     </joint>
-    <link name="vlp_lidar">
+    <link name="velodyne">
       <inertial>
         <mass value="0.1"/>
@@ -96,5 +96,29 @@
       </inertial>
     </link>
-    <!-- TODO, Add USB/Tier IV camera frames when camera integration is ready -->
+    <!-- USB cameras (TIER IV C1 via GMSL2-USB) — placeholder transforms; update after physical mounting -->
+    <xacro:macro name="usb_camera_frame" params="name">
+      <joint name="${name}_joint" type="fixed">
+        <origin
+          xyz="${calibration['sensor_kit_base_link'][name]['x']}
+               ${calibration['sensor_kit_base_link'][name]['y']}
+               ${calibration['sensor_kit_base_link'][name]['z']}"
+          rpy="${calibration['sensor_kit_base_link'][name]['roll']}
+               ${calibration['sensor_kit_base_link'][name]['pitch']}
+               ${calibration['sensor_kit_base_link'][name]['yaw']}"
+        />
+        <parent link="sensor_kit_base_link"/>
+        <child link="${name}"/>
+      </joint>
+      <link name="${name}">
+        <inertial>
+          <mass value="0.1"/>
+          <origin xyz="0 0 0"/>
+          <inertia ixx="0.1" ixy="0" ixz="0" iyy="0.1" iyz="0" izz="0.1"/>
+        </inertial>
+      </link>
+    </xacro:macro>
+    <xacro:usb_camera_frame name="usb_camera_left_optical_link"/>
+    <xacro:usb_camera_frame name="usb_camera_right_optical_link"/>
+    <xacro:usb_camera_frame name="usb_camera_rear_optical_link"/>
   </xacro:macro>
 </robot>

Commit message: feat(sensor_kit): anchor the ZED X to sensor_kit_base_link
Adds a zed_camera_link joint and its calibration entry. This is the one
ZED frame this project is responsible for placing - the threaded screw
hole in the camera's bottom face. Everything below it is fixed by the
camera's construction and comes from the vendor URDF, published by a
separate robot_state_publisher next to the driver.

Deliberately does not instantiate zed_macro.urdf.xacro here. Doing so
would republish camera_center and both lens chains that the driver-side
robot_state_publisher already provides, giving every one of those edges
two publishers.

The extrinsics are a placeholder of all zeros. They have to be measured
on the cart, to the screw hole - do not fold the lens offsets in, the
vendor URDF already applies them.

Co-Authored-By: Claude Opus 5 <noreply@anthropic.com>

File: golfcart_sensor_kit_description/urdf/sensor_kit.xacro (robot description, xacro)
@@ -136,4 +136,24 @@
     </joint>
     <link name="camera_right"/>
+    <!--
+      ZED X mounting point only. The camera's internal geometry
+      (zed_camera_center, the two lens frames, the optical frames) is published
+      by a separate robot_state_publisher in zed.launch.xml, fed the vendor's
+      zed_descr.urdf.xacro. Do not instantiate zed_macro here as well - that
+      would give every one of those edges two publishers.
+    -->
+    <joint name="zed_camera_joint" type="fixed">
+        <origin
+        xyz="${calibration['sensor_kit_base_link']['zed_camera_link']['x']}
+             ${calibration['sensor_kit_base_link']['zed_camera_link']['y']}
+             ${calibration['sensor_kit_base_link']['zed_camera_link']['z']}"
+        rpy="${calibration['sensor_kit_base_link']['zed_camera_link']['roll']}
+             ${calibration['sensor_kit_base_link']['zed_camera_link']['pitch']}
+             ${calibration['sensor_kit_base_link']['zed_camera_link']['yaw']}"
+            />
+        <parent link="sensor_kit_base_link"/>
+        <child link="zed_camera_link"/>
+    </joint>
+    <link name="zed_camera_link"/>
   </xacro:macro>
 </robot>

Commit message: feat(camera): give the GMSL cameras optical frames, and stamp them
The three cameras had one frame each, the point they are bolted at, with x
forward and y left like everything else on the vehicle. Image data was stamped
with it. Every projection is done in the optical convention -- x right, y down,
z along the view -- so anything taking CameraInfo at its word, which REP-103
says it should, came out rotated ninety degrees.

Each camera now has camera_NAME_optical_link as a fixed child of its mounting
frame, and the drivers stamp that instead. The rotation between them carries no
calibration and never changes; the mounting measurement stays where it belongs,
in the body frame, where sensor_kit_calibration.yaml can be read by someone
holding a tape measure.

Verified by expanding the description and walking the chain to base_link. For
all three cameras the optical frame now has image-down pointing down and the
view direction pointing out of the side its camera is on:

    camera_left_optical_link    right +forward   down -up   view +left
    camera_right_optical_link   right -forward   down -up   view -left
    camera_rear_optical_link    right +left      down -up   view -forward

This fixes the convention, not the calibration. The mounting values in
sensor_kit_calibration.yaml are still the round-number guesses phase 3A
describes, with roll and pitch hard-zeroed, so the frames are now correctly
shaped and still wrongly placed.

Co-Authored-By: Claude Opus 5 (1M context) <noreply@anthropic.com>
Claude-Session: https://claude.ai/code/session_01E3zgU7ETtbQXPomADLRM1T

File: golfcart_sensor_kit_description/urdf/sensor_kit.xacro (robot description, xacro)
@@ -96,5 +96,18 @@
       </inertial>
     </link>
-    <!-- USB/Tier IV camera -->
+    <!-- TIER IV GMSL cameras.
+         Each has two frames. The body frame, camera_NAME, is where the camera
+         is bolted and is what sensor_kit_calibration.yaml measures: x forward,
+         y left, z up, like every other frame on the vehicle. The optical
+         frame, camera_NAME_optical_link, is that same point turned into the
+         convention every projection uses (x right, y down, z along the view
+         direction), which is what REP-103 asks image data to be stamped with
+         and what the drivers now stamp. See camera_NAME.yaml.
+         Keeping both matters. A mounting measurement is taken in the body
+         frame and would be unreadable written optically; a projection is done
+         in the optical frame and comes out ninety degrees wrong if handed the
+         body one. The fixed rotation between them carries no calibration and
+         never changes.
+    -->
     <joint name="camera_left_joint" type="fixed">
         <origin
@@ -110,4 +123,10 @@
     </joint>
     <link name="camera_left"/>
+    <joint name="camera_left_optical_joint" type="fixed">
+        <origin xyz="0 0 0" rpy="${-pi/2} 0 ${-pi/2}"/>
+        <parent link="camera_left"/>
+        <child link="camera_left_optical_link"/>
+    </joint>
+    <link name="camera_left_optical_link"/>
     <joint name="camera_rear_joint" type="fixed">
         <origin
@@ -123,4 +142,10 @@
     </joint>
     <link name="camera_rear"/>
+    <joint name="camera_rear_optical_joint" type="fixed">
+        <origin xyz="0 0 0" rpy="${-pi/2} 0 ${-pi/2}"/>
+        <parent link="camera_rear"/>
+        <child link="camera_rear_optical_link"/>
+    </joint>
+    <link name="camera_rear_optical_link"/>
     <joint name="camera_right_joint" type="fixed">
         <origin
@@ -136,4 +161,10 @@
     </joint>
     <link name="camera_right"/>
+    <joint name="camera_right_optical_joint" type="fixed">
+        <origin xyz="0 0 0" rpy="${-pi/2} 0 ${-pi/2}"/>
+        <parent link="camera_right"/>
+        <child link="camera_right_optical_link"/>
+    </joint>
+    <link name="camera_right_optical_link"/>
     <!--
       ZED X mounting point only. The camera's internal geometry
